Commit message: added fk for each link in panda

File: panda.urdf (robot description, URDF)
Before this commit: robot panda, 12 links, 11 joints
Links:
- added link point1; visual box size=0.1 0.1 0.1
- added link point2; visual box size=0.1 0.1 0.1
- added link point3; visual box size=0.1 0.1 0.1
- added link point4; visual box size=0.1 0.1 0.1
- added link point5; visual box size=0.1 0.1 0.1
- added link point7; visual box size=0.1 0.1 0.1
- added link point8; visual box size=0.1 0.1 0.1
- link finger1: geometry collision mesh filename=../../../../research/projects/RMP2/src/models/panda/mesh/co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; visual mesh filename=../../../../research/projects/RMP2/src/models/panda/mesh/vi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
- link finger2: geometry collision mesh filename=../../../../research/projects/RMP2/src/models/panda/mesh/co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; visual mesh filename=../../../../research/projects/RMP2/src/models/panda/mesh/vi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
- link link0: geometry collision mesh filename=../../../../research/projects/RMP2/src/models/panda/mesh/co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; visual mesh filename=../../../../research/projects/RMP2/src/models/panda/mesh/vi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
- link link1: geometry collision mesh filename=../../../../research/projects/RMP2/src/models/panda/mesh/co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; visual mesh filename=../../../../research/projects/RMP2/src/models/panda/mesh/vi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
- link link2: geometry collision mesh filename=../../../../research/projects/RMP2/src/models/panda/mesh/co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; visual mesh filename=../../../../research/projects/RMP2/src/models/panda/mesh/vi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
- link link3: geometry collision mesh filename=../../../../research/projects/RMP2/src/models/panda/mesh/co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; visual mesh filename=../../../../research/projects/RMP2/src/models/panda/mesh/vi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
- link link4: geometry collision mesh filename=../../../../research/projects/RMP2/src/models/panda/mesh/co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; visual mesh filename=../../../../research/projects/RMP2/src/models/panda/mesh/vi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
- link link5: geometry collision mesh filename=../../../../research/projects/RMP2/src/models/panda/mesh/co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; visual mesh filename=../../../../research/projects/RMP2/src/models/panda/mesh/vi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
- link link6: geometry collision mesh filename=../../../../research/projects/RMP2/src/models/panda/mesh/co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; visual mesh filename=../../../../research/projects/RMP2/src/models/panda/mesh/vi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
- link link7: geometry collision mesh filename=../../../../research/projects/RMP2/src/models/panda/mesh/co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; visual mesh filename=../../../../research/projects/RMP2/src/models/panda/mesh/vi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
- link link8: geometry collision mesh filename=../../../../research/projects/RMP2/src/models/panda/mesh/co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; visual mesh filename=../../../../research/projects/RMP2/src/models/panda/mesh/vi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
Joints:
- added joint point1joint: type fixed, parent link1, child point1, origin xyz=0 0 -0.1 rpy=0 0 0
- added joint point2joint: type fixed, parent link2, child point2, origin xyz=0 -0.12 -0.0 rpy=0 0 0
- added joint point3joint: type fixed, parent link3, child point3, origin xyz=-0.0 -0.0 -0.05 rpy=0 0 0
- added joint point4joint: type fixed, parent link4, child point4, origin xyz=-0.0 0 -0.03 rpy=0 0 0
- added joint point5joint: type fixed, parent link5, child point5, origin xyz=0.0 0.0 -0.12 rpy=0 0 0
- added joint point7joint: type fixed, parent link7, child point7, origin xyz=0 0.0 0.0 rpy=0 0 0
- added joint point8joint: type fixed, parent link8, child point8, origin xyz=0 0.0 0.05 rpy=0 0 0
