Commit message: added arm contact points fk

File: arm.urdf (robot description, URDF)
Before this commit: robot prosthetic, 12 links, 11 joints
Links:
- added link point2; visual cylinder length=0.05 radius=0.05
- added link point3; visual cylinder length=0.05 radius=0.05
- added link point4; visual cylinder length=0.05 radius=0.05
- added link point5; visual cylinder length=0.05 radius=0.05
- added link point6; visual cylinder length=0.05 radius=0.05
- added link point7; visual cylinder length=0.05 radius=0.05
Joints:
- added joint point2joint: type fixed, parent link2, child point2, origin xyz=0 0 0 rpy=0 0 0
- added joint point3joint: type fixed, parent link3, child point3, origin xyz=0 0 0 rpy=0 0 0
- added joint point4joint: type fixed, parent link4, child point4, origin xyz=0 0 0.1 rpy=0 0 0
- added joint point5joint: type fixed, parent link4, child point5, origin xyz=0 0 -0.1 rpy=0 0 0
- added joint point7joint: type fixed, parent link6, child point6, origin xyz=0 0 0 rpy=0 0 0
- added joint point8joint: type fixed, parent link7, child point7, origin xyz=0 0 0 rpy=0 0 0
