Commit message: digit wholebody FK implemented

File: get_fkn_eqns/urdf/digit_model_mod.urdf (robot description, URDF)
Before this commit: robot digit, 31 links, 30 joints
Links:
- removed link left_wrist
- removed link right_wrist
- added link hcp, mass 0.005; collision box size=0.05 0.05 0.05; visual box size=0.15 0.15 0.15
- added link lcp0, mass 0.005; collision box size=0.05 0.05 0.05; visual box size=0.05 0.05 0.05
- added link lcp1, mass 0.005; collision box size=0.05 0.05 0.05; visual box size=0.05 0.05 0.05
- added link lcp2, mass 0.005; collision box size=0.05 0.05 0.05; visual box size=0.05 0.05 0.05
- added link lcp3, mass 0.005; collision box size=0.05 0.05 0.05; visual box size=0.05 0.05 0.05
- added link lcp4, mass 0.005; collision box size=0.05 0.05 0.05; visual box size=0.05 0.05 0.05
- added link lcp5, mass 0.005; collision box size=0.05 0.05 0.05; visual box size=0.05 0.05 0.05
- added link lcp6, mass 0.005; collision box size=0.05 0.05 0.05; visual box size=0.05 0.05 0.05
- added link lcp7, mass 0.005; collision box size=0.05 0.05 0.05; visual box size=0.05 0.05 0.05
- added link rcp0, mass 0.005; collision box size=0.05 0.05 0.05; visual box size=0.05 0.05 0.05
- added link rcp1, mass 0.005; collision box size=0.05 0.05 0.05; visual box size=0.05 0.05 0.05
- added link rcp2, mass 0.005; collision box size=0.05 0.05 0.05; visual box size=0.05 0.05 0.05
- added link rcp3, mass 0.005; collision box size=0.05 0.05 0.05; visual box size=0.05 0.05 0.05
- added link rcp4, mass 0.005; collision box size=0.05 0.05 0.05; visual box size=0.05 0.05 0.05
- added link rcp5, mass 0.005; collision box size=0.05 0.05 0.05; visual box size=0.05 0.05 0.05
- added link rcp6, mass 0.005; collision box size=0.05 0.05 0.05; visual box size=0.05 0.05 0.05
- added link rcp7, mass 0.005; collision box size=0.05 0.05 0.05; visual box size=0.05 0.05 0.05
Joints:
- removed joint elbow_joint_left
- removed joint elbow_joint_right
- removed joint hip_abduction_left
- removed joint hip_abduction_right
- removed joint hip_flexion_left
- removed joint hip_flexion_right
- removed joint hip_rotation_left
- removed joint hip_rotation_right
- removed joint knee_joint_left
- removed joint knee_joint_right
- removed joint knee_to_shin_left
- removed joint knee_to_shin_right
- removed joint shin_to_tarsus_left
- removed joint shin_to_tarsus_right
- removed joint shoulder_pitch_joint_left
- removed joint shoulder_pitch_joint_right
- removed joint shoulder_roll_joint_left
- removed joint shoulder_roll_joint_right
- removed joint shoulder_yaw_joint_left
- removed joint shoulder_yaw_joint_right
- removed joint toe_pitch_joint_left
- removed joint toe_pitch_joint_right
- removed joint toe_roll_joint_left
- removed joint toe_roll_joint_right
- added joint LeftElbow: type continuous, parent left_shoulder_yaw, child left_elbow, origin xyz=0 -0.0385 0.185 rpy=1.57079632679 -0.3926991 0, axis 0 0 1, limit lower=-1.3526 upper=1.3526 effort=1.4 velocity=12.5
- added joint LeftHipPitch: type continuous, parent left_hip_yaw, child left_hip_pitch, origin xyz=0 0.004 0.068 rpy=-1.57079632679 -0.785398163397 3.14159265359, axis 0 0 -1, limit lower=-1.0472 upper=1.57079632679 effort=12.5 velocity=8.5
- added joint LeftHipRoll: type continuous, parent torso, child left_hip_roll, origin xyz=-0.001 0.091 0 rpy=1.57079632679 -1.1955506 -1.57079632679, axis 0 0 1, limit lower=-1.0472 upper=1.0472 effort=1.4 velocity=12.15
- added joint LeftHipYaw: type continuous, parent left_hip_roll, child left_hip_yaw, origin xyz=-0.0505 0 0.044 rpy=0 -1.57079632679 0, axis 0 0 1, limit lower=-0.698132 upper=0.698132 effort=1.4 velocity=12.15
- added joint LeftKnee: type continuous, parent left_hip_pitch, child left_knee, origin xyz=0.12 0 0.0045 rpy=0 0 -1.57079632679, axis 0 0 1, limit lower=-1.2392 upper=0.8727 effort=12.5 velocity=8.5085
- added joint LeftShin: type continuous, parent left_knee, child left_shin, origin xyz=0.060677 0.047406 0 rpy=0 0 0, axis 0 0 1, limit lower=-0.35 upper=0.35 effort=0 velocity=10
- added joint LeftShoulderPitch: type continuous, parent left_shoulder_roll, child left_shoulder_pitch, origin xyz=-0.00317 -0.011055 0.0555 rpy=1.57079632679 0.785398163397 -0.2792527, axis 0 0 -1, limit lower=-2.5307 upper=2.5307 effort=1.4 velocity=12.5
- added joint LeftShoulderRoll: type continuous, parent torso, child left_shoulder_roll, origin xyz=-0.001 0.12 0.4 rpy=-1.57079632679 -1.3962633 1.57079632679, axis 0 0 1, limit lower=-1.309 upper=1.309 effort=1.4 velocity=12.5
- added joint LeftShoulderYaw: type continuous, parent left_shoulder_pitch, child left_shoulder_yaw, origin xyz=0 -0.165 -0.1 rpy=1.57079632679 0 0, axis 0 0 1, limit lower=-1.7453 upper=1.7453 effort=1.4 velocity=10
- added joint LeftTarsus: type continuous, parent left_shin, child left_tarsus, origin xyz=0.434759 0.02 0 rpy=0 0 1.7976891, axis 0 0 1, limit lower=-0.8779 upper=1.2497 effort=0 velocity=20
- added joint LeftToePitch: type continuous, parent left_tarsus, child left_toe_pitch, origin xyz=0.408 -0.04 0 rpy=0 0 1.1956, axis 0 0 1, limit lower=-0.785398163397 upper=0.785398163397 effort=0.9 velocity=11.5
- added joint LeftToeRoll: type continuous, parent left_toe_pitch, child left_toe_roll, origin xyz=0 0 0 rpy=0 1.57079632679 0, axis 0 0 1, limit lower=-0.6109 upper=0.6109 effort=0.9 velocity=11.5
- added joint RightElbow: type continuous, parent right_shoulder_yaw, child right_elbow, origin xyz=0 0.0385 0.185 rpy=-1.57079632679 -0.3926991 0, axis 0 0 1, limit lower=-1.3526 upper=1.3526 effort=1.4 velocity=12.5
- added joint RightHipPitch: type continuous, parent right_hip_yaw, child right_hip_pitch, origin xyz=0 -0.004 0.068 rpy=1.57079632679 -0.785398163397 -3.14159265359, axis 0 0 -1, limit lower=-1.57079632679 upper=1.0472 effort=12.5 velocity=8.5
- added joint RightHipRoll: type continuous, parent torso, child right_hip_roll, origin xyz=-0.001 -0.091 0 rpy=-1.57079632679 -1.1955506 1.57079632679, axis 0 0 1, limit lower=-1.0472 upper=1.0472 effort=1.4 velocity=12.15
- added joint RightHipYaw: type continuous, parent right_hip_roll, child right_hip_yaw, origin xyz=-0.0505 0 0.044 rpy=0 -1.57079632679 0, axis 0 0 1, limit lower=-0.698132 upper=0.698132 effort=1.4 velocity=12.15
- added joint RightKnee: type continuous, parent right_hip_pitch, child right_knee, origin xyz=0.12 0 0.0045 rpy=0 0 1.57079632679, axis 0 0 1, limit lower=-0.8727 upper=1.2392 effort=12.5 velocity=8.5085
- added joint RightShin: type continuous, parent right_knee, child right_shin, origin xyz=0.060677 -0.047406 0 rpy=0 0 0, axis 0 0 1, limit lower=-0.35 upper=0.35 effort=0 velocity=10
- added joint RightShoulderPitch: type continuous, parent right_shoulder_roll, child right_shoulder_pitch, origin xyz=-0.00317 0.011055 0.0555 rpy=-1.57079632679 0.785398163397 0.2792527, axis 0 0 -1, limit lower=-2.5307 upper=2.5307 effort=1.4 velocity=12.5
- added joint RightShoulderRoll: type continuous, parent torso, child right_shoulder_roll, origin xyz=-0.001 -0.12 0.4 rpy=1.57079632679 -1.3962633 -1.57079632679, axis 0 0 1, limit lower=-1.309 upper=1.309 effort=1.4 velocity=12.5
- added joint RightShoulderYaw: type continuous, parent right_shoulder_pitch, child right_shoulder_yaw, origin xyz=0 0.165 -0.1 rpy=-1.57079632679 0 0, axis 0 0 1, limit lower=-1.7453 upper=1.7453 effort=1.4 velocity=10
- added joint RightTarsus: type continuous, parent right_shin, child right_tarsus, origin xyz=0.434759 -0.02 0 rpy=0 0 -1.7976891, axis 0 0 1, limit lower=-1.2497 upper=0.8779 effort=0 velocity=20
- added joint RightToePitch: type continuous, parent right_tarsus, child right_toe_pitch, origin xyz=0.408 0.04 0 rpy=0 0 -1.1956, axis 0 0 1, limit lower=-0.785398163397 upper=0.785398163397 effort=0.9 velocity=11.5
- added joint RightToeRoll: type continuous, parent right_toe_pitch, child right_toe_roll, origin xyz=0 0 0 rpy=0 1.57079632679 0, axis 0 0 1, limit lower=-0.6109 upper=0.6109 effort=0.9 velocity=11.5
- added joint hcpjoint: type fixed, parent torso, child hcp, origin xyz=0.0 0.0 0.5 rpy=0.0 0.0 0.0
- added joint lcp1joint: type fixed, parent left_elbow, child lcp1, origin xyz=0.22 0.0 -0.04 rpy=0.0 0.0 0.0
- added joint lcp2joint: type fixed, parent left_shoulder_yaw, child lcp2, origin xyz=0.0 0.0 0.2 rpy=0.0 0.0 0.0
- added joint lcp3joint: type fixed, parent left_shoulder_yaw, child lcp3, origin xyz=0.0 0.0 0.0 rpy=0.0 0.0 0.0
- added joint lcp4joint: type fixed, parent left_hip_pitch, child lcp4, origin xyz=0.08 0 -0.05 rpy=0.0 0.0 0.0
- added joint lcp5joint: type fixed, parent left_knee, child lcp5, origin xyz=0.25 0.05 0.0 rpy=0.0 0.0 0.0
- added joint lcp6joint: type fixed, parent left_tarsus, child lcp6, origin xyz=0.2 -0.025 0.0 rpy=0.0 0.0 0.0
- added joint lcp7joint: type fixed, parent left_toe_pitch, child lcp7, origin xyz=-0.05 -0.01 0.0 rpy=0.0 0.0 -0.523
- added joint rcp1joint: type fixed, parent right_elbow, child rcp1, origin xyz=0.22 0.0 -0.04 rpy=0.0 0.0 0.0
- added joint rcp2joint: type fixed, parent right_shoulder_yaw, child rcp2, origin xyz=0.0 0.0 0.2 rpy=0.0 0.0 0.0
- added joint rcp3joint: type fixed, parent right_shoulder_yaw, child rcp3, origin xyz=0.0 0.0 0.0 rpy=0.0 0.0 0.0
- added joint rcp4joint: type fixed, parent right_hip_pitch, child rcp4, origin xyz=0.08 0 -0.05 rpy=0.0 0.0 0.0
- added joint rcp5joint: type fixed, parent right_knee, child rcp5, origin xyz=0.25 -0.05 0.0 rpy=0.0 0.0 0.0
- added joint rcp6joint: type fixed, parent right_tarsus, child rcp6, origin xyz=0.2 0.025 0.0 rpy=0.0 0.0 0.0
- added joint rcp7joint: type fixed, parent right_toe_pitch, child rcp7, origin xyz=-0.05 -0.01 0.0 rpy=0.0  0.0 0.523
- joint wrist_joint_left: child left_wrist -> lcp0
- joint wrist_joint_right: child right_wrist -> rcp0
